Commit message: twip sim tuning

File: urdf/robot.urdf.xacro (robot description, xacro)
@@ -1,4 +1,4 @@
 <?xml version="1.0"?>
-<robot xmlns:xacro="http://www.ros.org/wiki/xacro"  name="bi_pedal_a1">
+<robot xmlns:xacro="http://www.ros.org/wiki/xacro"  name="twip">
     <!-- <xacro:arg name="cmd_mode" default="position"/>
     <xacro:arg name="HW_mode" default="mock"/> -->

File: urdf/robot_core.xacro (robot description, xacro)
@@ -83,5 +83,5 @@
         <child link="right_wheel_link"/>
         <origin xyz="-0.084 0 0" rpy="0 ${-pi/2} 0"/>
-        <axis xyz="0 0 1"/>
+        <axis xyz="0 0 -1"/>
     </joint>
 </robot>
